File: switchboard 2.brd (EAGLE design)
At the start: 100 x 60 mm, 189 parts, among them IC1 MT8816AP, IC11 LMV321M5, IC12 74HC595D, IC14 74LVC1G125DBV, IC15 74LVC1G125DBV, IC16 LM2940, IC17 PC817S OPTO, IC18 Z8F2480SO, IC19 Z8F042A, IC2 NE5532D, IC3 TC7660-SOIC, IC4 TC7660-SOIC, IC5 FT232RL, IC6 78L05F, IC7 LD117AS33TR, IC8 SPI_MEMORY-SOIC, IC9 NE5532D, X1 MINI-USB-SCHIELD-32005-301

Commit message: MCU Z8F082 dropped. Bidirectional MOSFET level shifter added. Reset signal added on debug connector.
Parts:
- removed IC19: Z8F042A, Maxwell_Bohr:SSOP28
- removed MNT1: (no value), con-lstb:MA03-2
- removed R_DBG: 10k, rcl:R0603
- added JP21, JP22, JP23, JP25: (no value), pinhead:1X02
- added JP24: (no value), pinhead:2X03
- added Q1, Q2: 2N7002, PATSKO:SOT23
- added R54, R55: 10k, rcl:R0603
- added R56, R57, R58: 10k, rcl:R0805
- added R59: 10k SMD, rcl:R0603
- R20: value 1k -> 10k
- moved C4 802.3 mm to (-261.0, -720.1), flipped to the top, turned to 0 degrees
- moved JP9 375.6 mm to (36.2, 3.81), turned to 90 degrees
- moved JP8 369.1 mm to (33.0, 3.81), turned to 90 degrees
- moved JP7 362.6 mm to (29.8, 3.81), turned to 90 degrees
- moved JP1 31.6 mm to (11.1, 3.49), turned to 90 degrees
- moved JP11 18.5 mm to (11.4, 29.2)
- moved JP6 13.0 mm to (26.7, 3.81), turned to 90 degrees
- moved JP5 9.86 mm to (23.5, 3.81), turned to 90 degrees
- moved JP4 6.84 mm to (20.3, 3.81), turned to 90 degrees
- moved JP3 3.70 mm to (17.1, 3.81)
- moved JP2 1.42 mm to (14.0, 3.81)
Connections:
- removed net CLOCK: IC19.12
- removed net CS_SWITCH: IC1.40, IC18.21
- removed net C_SW1: IC1.5, IC18.23, R9.2
- removed net DATA: IC19.11
- removed net ENABLE: IC19.15
- removed net MCU_SW1: IC19.23
- removed net MCU_SW2: IC19.24
- removed net MCU_SW3: IC19.25
- removed net MCU_SW4: IC19.26
- removed net MCU_SW5: IC19.16
- removed net MCU_SW6: IC19.17
- removed net XIN: IC19.7
- removed net XOUT: IC19.8
- removed net XP_DBG: IC18.22, IC19.22, MNT1.4, R_DBG.2
- removed net XP_RST: IC19.21
- new net BTN6/C_SW1: IC1.5, IC18.8, JP21.2, JP22.2, JP23.2, R59.2
- new net CS_SWITCH/AD0: IC1.40, IC11.3, IC11.4, IC18.27, R56.1
- new net DBG: IC18.22, JP24.4, R55.2
- new net MOSI_5V: IC1.42, Q2.3, R58.1
- new net RST: C4.1, IC18.21, JP24.6, JP25.1
- new net SCK_5V: IC1.20, Q1.3, R57.1
- net +3V3: now also JP24.1, Q1.1, Q2.1, R55.1; no longer C4.1, IC19.5, IC19.6, MNT1.1, R_DBG.1
- net +5V: now also R56.2, R57.2, R58.2, R59.1
- net 5V_USB: now also R54.1
- net AD0: no longer IC11.3, IC11.4, IC18.27, IC19.27
- net BTN0: now also JP23.1; no longer IC19.28
- net BTN1: now also JP22.1; no longer IC19.1
- net BTN2: now also JP21.1; no longer IC19.4
- net BTN3: no longer IC19.2
- net BTN4: no longer IC19.3
- net BTN5: no longer IC19.18
- net CS_MEM: now also IC18.25; no longer IC18.8
- net CS_SHIFT: now also IC18.26; no longer IC18.19
- net C_SW2: now also IC18.11; no longer IC18.15
- net C_SW3: now also IC18.15; no longer IC18.25
- net C_SW4: now also IC18.18; no longer IC18.26
- net C_SW5: now also IC18.23; no longer IC18.11
- net C_SW6: now also IC18.19; no longer IC18.18
- net C_SW7: now also R9.2
- net EIN_2: now also IC1.34
- net EIN_3: now also IC1.33
- net EIN_4: now also IC1.32
- net EIN_5: now also IC1.9
- net EIN_6: now also IC1.10
- net EIN_7: now also IC1.11
- net EIN_8: now also IC1.12
- net GND: now also JP24.3, JP24.5, JP25.2; no longer IC19.10, IC19.9, MNT1.3, MNT1.5
- net MOSI: now also Q2.2; no longer IC1.42
- net SCK: now also Q1.2; no longer IC1.20
- net UART_RX: no longer IC19.13
- net UART_TX: no longer IC19.14
- net USB_DETECT: now also R54.2
Routing:
- net XP_DBG: track 14.3 -> 0.00 mm
- net XOUT: track 11.5 -> 0.00 mm
- net XIN: track 11.5 -> 0.00 mm
- net DBG: track 0.00 -> 10.2 mm
- net AD0: track 9.03 -> 0.00 mm
- net CS_SWITCH/AD0: track 0.00 -> 9.00 mm
- net +3V3: track 28.0 -> 21.5 mm
- net MCU_SW6: track 5.33 -> 0.00 mm
- net MCU_SW5: track 5.28 -> 0.00 mm
- net C_SW4: track 5.18 -> 0.00 mm
- net CS_SHIFT: track 0.00 -> 5.18 mm
- net BTN5: track 5.16 -> 0.00 mm
- net ENABLE: track 5.14 -> 0.00 mm
- net MCU_SW4: track 4.92 -> 0.00 mm
- net MCU_SW2: track 4.79 -> 0.00 mm
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
Commit message: General revisions and mods to the schematic - series resistors added to UART_RX, 3.3V selection jumper removed, USB_DETECT zener removed. Spark gaps added at audio inputs and outputs.
Parts:
- removed D8: 3V3 ZENER, diode:SOD80C
- removed IC18: Z8F2480SO, LUIS:SO28W
- removed SJ4: (no value), jumper:SJ_2
- added IC10: Z8F2480SO, PATSKO:SO28W
- added R60: 1k SMD, rcl:R0805
- added R71: 1k, rcl:R0603
- added U$5, U$6, U$7, U$8: SPARK_GAP, PATSKO:SPARK-GAP-8
Connections:
- removed net 3V3_FTDI: C33.1, IC5.17, SJ4.3
- removed net 3V3_REG: C32.+, IC7.4, SJ4.1
- new net N$35: IC5.1, R71.1
- net +3V3: now also C32.+, C33.1, IC10.5, IC10.6, IC5.17, IC7.4; no longer IC18.5, IC18.6, SJ4.2
- net BTN0: now also IC10.28; no longer IC18.28
- net BTN1: now also IC10.1; no longer IC18.1
- net BTN2: now also IC10.4; no longer IC18.4
- net BTN3: now also IC10.2; no longer IC18.2
- net BTN4: now also IC10.3; no longer IC18.3
- net BTN5: now also IC10.7; no longer IC18.7
- net BTN6/C_SW1: now also IC10.8; no longer IC18.8
- net CS_MEM: now also IC10.25; no longer IC18.25
- net CS_SHIFT: now also IC10.26; no longer IC18.26
- net CS_SWITCH/AD0: now also IC10.27; no longer IC18.27
- net C_SW2: now also IC10.11; no longer IC18.11
- net C_SW3: now also IC10.15; no longer IC18.15
- net C_SW4: now also IC10.18; no longer IC18.18
- net C_SW5: now also IC10.23; no longer IC18.23
- net C_SW6: now also IC10.19; no longer IC18.19
- net C_SW7: now also IC10.20; no longer IC18.20
- net DBG: now also IC10.22; no longer IC18.22
- net GND: now also IC10.10, IC10.9, U$5.P$2, U$6.P$2, U$7.P$2, U$8.P$2; no longer D8.A, IC18.10, IC18.9
- net INPUT1: now also U$5.P$1
- net INPUT2: now also U$6.P$1
- net MISO: now also IC10.24; no longer IC18.24
- net MOSI: now also IC10.16; no longer IC18.16
- net OUTPUT1: now also U$7.P$1
- net OUTPUT2: now also U$8.P$1
- net RST: now also IC10.21; no longer IC18.21
- net SCK: now also IC10.17; no longer IC18.17
- net UART_RX: now also IC10.13, R60.1, R60.2, R71.2; no longer IC18.13, IC5.1
- net UART_TX: now also IC10.14; no longer IC18.14
- net USB_DETECT: now also IC10.12; no longer D8.C, IC18.12
Routing:
- net +3V3: track 21.5 -> 5.61 mm
- net DBG: track 10.2 -> 0.00 mm
- net BTN0: track 9.79 -> 0.00 mm
- net CS_SWITCH/AD0: track 9.00 -> 0.00 mm
- net BTN1: track 7.12 -> 0.00 mm
- net BTN4: track 5.92 -> 0.00 mm
- net BTN3: track 5.65 -> 0.00 mm
- net BTN2: track 5.23 -> 0.00 mm
- net CS_SHIFT: track 5.18 -> 0.00 mm
- net C_SW5: track 3.90 -> 0.00 mm
- net CS_MEM: track 3.38 -> 0.00 mm
