File: switchboard 2.brd (EAGLE design)
At the start: 100 x 60 mm, 214 parts, among them IC1 MT8816AP, IC10 Z8F2480SO, IC11 LMV321M5, IC12 74HC595D, IC14 74LVC1G125DBV, IC15 74LVC1G125DBV, IC16 LM2940-9, IC17 PC817S OPTO, IC2 NE5532D, IC3 TC7660-SOIC, IC4 TC7660-SOIC, IC5 FT232RL, IC6 78L05F, IC7 LD117AS33TR, IC8 SPI_MEMORY-SOIC, IC9 NE5532D, Q3 FDN352AP, X1 MINI-USB-SCHIELD-32005-301

Commit message: Layout development. Minor component name and package changes.
Parts:
- removed JP1, JP2, JP3: (no value), pinhead-2:2X03SMD
- removed JP10, JP15, JP26, JP27, JP28: (no value), pinhead-2:2X06SMD
- removed JP11: (no value), pinhead:1X05
- removed JP18: (no value), pinhead:1X10
- removed JP24: (no value), pinhead:2X03
- removed P_OUT1: (no value), pinhead:1X02
- added JP_AUDIOEFF1, JP_AUDIOEFF2, JP_AUDIOEFF3, JP_BTNS1, JP_BTNS2: (no value), pinhead-2:2X06SMD
- added JP_DBG: (no value), pinhead:2X03
- added JP_OUTS1: (no value), pinhead:1X10
- added JP_POWEREFF1, JP_POWEREFF2, JP_POWEREFF3: (no value), pinhead-2:2X03SMD
- added JP_USB: (no value), pinhead:1X05
- added P_OUT2: (no value), pinhead:1X02
- C10, C11, C2, C6: device rcl:E2,5-6 -> PATSKO:SMB-SMA-0805-0603
- C30: device rcl:C0805 -> rcl:C0603
- moved P_UART 1114.8 mm to (92.7, 63.5)
- moved C6 1097.5 mm to (-320.0, -991.9), turned to 0 degrees
- moved R80 1001.5 mm to (11.4, 24.1), flipped to the bottom
- moved R79 1000.6 mm to (11.4, 21.6), flipped to the bottom
- moved R78 991.9 mm to (11.4, 19.1), flipped to the bottom
- moved R77 991.1 mm to (11.4, 16.5), flipped to the bottom
- moved P_I2C 990.4 mm to (94.0, 73.7)
- moved R75 977.9 mm to (7.62, 8.89), flipped to the bottom, turned to 270 degrees
- moved R76 977.1 mm to (10.2, 8.89), flipped to the bottom, turned to 270 degrees
- moved Q3 974.9 mm to (91.4, 41.9), turned to 180 degrees
- moved P_SPI 973.0 mm to (92.7, 71.1)
- moved R74 972.7 mm to (15.2, 7.62), flipped to the bottom
- moved R59 972.5 mm to (24.1, 7.62), flipped to the bottom, turned to 90 degrees
- moved R56 972.5 mm to (44.5, 10.2), flipped to the bottom, turned to 90 degrees
- moved R73 971.9 mm to (15.2, 5.08), flipped to the bottom
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Connections:
- new net N$77: C43.2, R77.2
- new net N$78: C41.2, R75.2
- new net N$79: C42.2, R76.2
- new net N$80: C44.2, R78.2
- new net N$81: C45.2, R79.2
- new net N$82: C46.2, R80.2
- net +18V: now also JP_POWEREFF1.5, JP_POWEREFF1.6, JP_POWEREFF2.5, JP_POWEREFF2.6, JP_POWEREFF3.5, JP_POWEREFF3.6; no longer JP1.5, JP1.6, JP2.5, JP2.6, JP3.5, JP3.6
- net +3V3: now also JP_DBG.1; no longer JP24.1
- net +9V: now also JP_POWEREFF1.1, JP_POWEREFF1.2, JP_POWEREFF2.1, JP_POWEREFF2.2, JP_POWEREFF3.1, JP_POWEREFF3.2; no longer JP1.1, JP1.2, JP2.1, JP2.2, JP3.1, JP3.2
- net BTN0: now also JP_BTNS1.1, JP_BTNS1.7, JP_BTNS2.1, JP_BTNS2.7; no longer JP10.1, JP10.7, JP15.1, JP15.7
- net BTN1: now also JP_BTNS1.3, JP_BTNS1.9, JP_BTNS2.3, JP_BTNS2.9; no longer JP10.3, JP10.9, JP15.3, JP15.9
- net BTN2: now also JP_BTNS1.11, JP_BTNS1.5, JP_BTNS2.11, JP_BTNS2.5; no longer JP10.11, JP10.5, JP15.11, JP15.5
- net BTN3: now also JP_BTNS1.2, JP_BTNS1.4, JP_BTNS1.6; no longer JP10.2, JP10.4, JP10.6
- net BTN4: now also JP_BTNS1.10, JP_BTNS1.12, JP_BTNS1.8; no longer JP10.10, JP10.12, JP10.8
- net BTN5: now also JP_BTNS2.2, JP_BTNS2.4, JP_BTNS2.6; no longer JP15.2, JP15.4, JP15.6
- net BTN6/C_SW1: now also JP_BTNS2.10, JP_BTNS2.12, JP_BTNS2.8; no longer JP15.10, JP15.12, JP15.8
- net D+: now also JP_USB.3; no longer JP11.3
- net D-: now also JP_USB.4; no longer JP11.4
- net DBG: now also JP_DBG.4; no longer JP24.4
- net GND: now also JP_AUDIOEFF1.10, JP_AUDIOEFF1.12, JP_AUDIOEFF1.2, JP_AUDIOEFF1.4, JP_AUDIOEFF1.6, JP_AUDIOEFF1.8, JP_AUDIOEFF2.10, JP_AUDIOEFF2.12, JP_AUDIOEFF2.2, JP_AUDIOEFF2.4, JP_AUDIOEFF2.6, JP_AUDIOEFF2.8, JP_AUDIOEFF3.10, JP_AUDIOEFF3.12, JP_AUDIOEFF3.2, JP_AUDIOEFF3.4, JP_AUDIOEFF3.6, JP_AUDIOEFF3.8, JP_DBG.3, JP_DBG.5, JP_OUTS1.9, JP_POWEREFF1.3, JP_POWEREFF1.4, JP_POWEREFF2.3, JP_POWEREFF2.4, JP_POWEREFF3.3, JP_POWEREFF3.4, JP_USB.2, P_OUT2.2; no longer JP1.3, JP1.4, JP11.2, JP18.9, JP2.3, JP2.4, JP24.3, JP24.5, JP26.10, JP26.12, JP26.2, JP26.4, JP26.6, JP26.8, JP27.10, JP27.12, JP27.2, JP27.4, JP27.6, JP27.8, JP28.10, JP28.12, JP28.2, JP28.4, JP28.6, JP28.8, JP3.3, JP3.4, P_OUT1.2
- net N$12: now also JP_AUDIOEFF1.1; no longer JP27.1
- net N$14: now also C10.-; no longer C6.-
- net N$19: now also JP_AUDIOEFF1.11; no longer JP27.11
- net N$21: now also JP_AUDIOEFF3.1; no longer JP26.1
- net N$27: now also C6.+; no longer C10.+
- net N$32: now also JP_AUDIOEFF3.3; no longer JP26.3
- net N$36: now also JP_OUTS1.1; no longer JP18.1
- net N$37: now also JP_OUTS1.2; no longer JP18.2
- net N$38: now also JP_OUTS1.3; no longer JP18.3
- net N$39: now also JP_OUTS1.4; no longer JP18.4
- net N$40: now also JP_OUTS1.5; no longer JP18.5
- net N$41: now also JP_OUTS1.6; no longer JP18.6
- net N$42: now also JP_OUTS1.7; no longer JP18.7
- net N$43: now also JP_OUTS1.8; no longer JP18.8
- net N$44: now also JP_OUTS1.10; no longer JP18.10
- net N$52: now also JP_AUDIOEFF3.5; no longer JP26.5
- net N$53: now also JP_AUDIOEFF3.7; no longer JP26.7
- net N$54: now also C6.-; no longer C10.-
- net N$59: now also JP_AUDIOEFF3.9; no longer JP26.9
- net N$62: now also JP_AUDIOEFF3.11; no longer JP26.11
- net N$64: now also JP_AUDIOEFF2.11; no longer JP28.11
- net N$69: now also JP_AUDIOEFF1.3; no longer JP27.3
- net N$70: now also JP_AUDIOEFF1.9; no longer JP27.9
- net N$71: now also JP_AUDIOEFF1.7; no longer JP27.7
- net N$72: now also JP_AUDIOEFF1.5; no longer JP27.5
- net N$73: now also JP_AUDIOEFF2.3; no longer JP28.3
- net N$74: now also JP_AUDIOEFF2.9; no longer JP28.9
- net N$75: now also JP_AUDIOEFF2.5; no longer JP28.5
- net N$76: now also JP_AUDIOEFF2.7; no longer JP28.7
- net N$8: now also C10.+; no longer C6.+
- net N$9: now also JP_AUDIOEFF2.1; no longer JP28.1
- net OUTPUT2: now also P_OUT2.1; no longer P_OUT1.1
- net RST: now also JP_DBG.6; no longer JP24.6
- net USB_SHLD: now also JP_USB.1; no longer JP11.1
- net VIN_USB: now also JP_USB.5; no longer JP11.5
Routing:
- net SWOUT_1: track 42.7 -> 0.00 mm, vias 2 -> 0
- net SW_IN_1: track 23.0 -> 0.00 mm, vias 2 -> 0
- net N$20: track 15.0 -> 0.00 mm
- net N$3: track 14.5 -> 0.00 mm
- net N$31: track 11.1 -> 0.00 mm
- net N$14: track 10.5 -> 0.00 mm
- net N$28: track 10.2 -> 0.00 mm
- net N$4: track 10.1 -> 0.00 mm
- net N$30: track 9.94 -> 0.00 mm
- net +9V: track 9.64 -> 0.00 mm
- net N$29: track 8.67 -> 0.00 mm
- net N$26: track 7.40 -> 0.00 mm
- net N$10: track 6.52 -> 0.00 mm
- net N$22: track 6.13 -> 0.00 mm
- net N$24: track 6.10 -> 0.00 mm
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